File: hw/fanctl.sch (KiCad schematic (older format))
At the start: 34 parts, among them Q0 Q_PMOS_SDG, U0 ULN2003A

Commit message: Some updates
Parts:
- added SW?: SW_PUSH, symbol SW_PUSH
Connections:
- wire segments 123 -> 128
Changed lines of the file:
@@
 LIBS:contrib
 LIBS:valves
+LIBS:fanctl-cache
 EELAYER 25 0
 EELAYER END
@@
 Wire Wire Line
 	3950 2700 3100 2700
+$Comp
+L GND #PWR?
+U 1 1 566C5775
+P 5300 7300
+F 0 "#PWR?" H 5300 7050 50  0001 C CNN
+F 1 "GND" H 5300 7150 50  0000 C CNN
+F 2 "" H 5300 7300 50  0000 C CNN
+F 3 "" H 5300 7300 50  0000 C CNN
+	1    5300 7300
+	1    0    0    -1
+$EndComp
+Wire Wire Line
+	5100 7300 5300 7300
+$Comp
+L GND #PWR?
+U 1 1 566C5998
+P 1300 5600
+F 0 "#PWR?" H 1300 5350 50  0001 C CNN
+F 1 "GND" H 1300 5450 50  0000 C CNN
+F 2 "" H 1300 5600 50  0000 C CNN
+F 3 "" H 1300 5600 50  0000 C CNN
+	1    1300 5600
+	1    0    0    -1
+$EndComp
+Wire Wire Line
+	1150 5750 1150 5600
+Wire Wire Line
+	1150 5600 1300 5600
+$Comp
+L SW_PUSH SW?
+U 1 1 566C5FF7
+P 4650 4700
+F 0 "SW?" H 4800 4810 50  0000 C CNN
+F 1 "SW_PUSH" H 4650 4620 50  0000 C CNN
+F 2 "" H 4650 4700 50  0000 C CNN
+F 3 "" H 4650 4700 50  0000 C CNN
+	1    4650 4700
+	1    0    0    -1
+$EndComp
+Wire Wire Line
+	4350 5400 4350 4700
+$Comp
+L GND #PWR?
+U 1 1 566C6164
+P 5050 4700
+F 0 "#PWR?" H 5050 4450 50  0001 C CNN
+F 1 "GND" H 5050 4550 50  0000 C CNN
+F 2 "" H 5050 4700 50  0000 C CNN
+F 3 "" H 5050 4700 50  0000 C CNN
+	1    5050 4700
+	0    -1   -1   0
+$EndComp
+Wire Wire Line
+	5050 4700 4950 4700
 $EndSCHEMATC

Commit message: Updates
Parts:
- added D? (x2): ZENER, symbol ZENER
- added R? (x2): R, symbol R
Connections:
- wire segments 128 -> 142

Commit message: Changes
Parts:
- removed R? (x14): R, symbol R
- removed SW?: SW_PUSH, symbol SW_PUSH
- added JP0: JUMPER, symbol JUMPER
- added R0: 1.5k, symbol R
- added R1: 68, symbol R
- added R? (x12): R, symbol R
- D? (x2): symbol ZENER -> ZENER-RESCUE-fanctl
- gave numbers to parts that had none: 5
- renumbered JP0 to JP1
Connections:
- wire segments 142 -> 143

Commit message: Changes
Parts:
- added C0: 0.1uF, symbol C
- added R?: R, symbol R
Connections:
- net GND: now also C0.1; no longer D?.1 (A), P?.2 (P2), P?.3 (P3), P?.4 (GND), P?.5 (shield)
- net at IC?.20 (AVCC): now also IC?.7 (VCC), P?.1 (VCC), R0.2, C0.2
- net at IC?.3 ((PCINT17/TXD)PD1): now also R?.1
- net at D?.2 (K), P?.3 (D+): now also R?.2
- new net: D?.1 (A), P?.2 (P2), P?.3 (P3), P?.5 (shield)
- no-connect marks 1 -> 2
Changed lines of the file:
@@
 EESchema Schematic File Version 2
-LIBS:fanctl-rescue
 LIBS:power
 LIBS:device
@@
 	2050 5750 2050 5950
 Connection ~ 1150 5350
-Wire Wire Line
-	1150 5750 1150 5350
-Wire Wire Line
-	600  5200 600  5350
-Wire Wire Line
-	600  5350 1700 5350
 Connection ~ 1400 5950
 Wire Wire Line
@@
 Wire Wire Line
 	2050 5950 1150 5950
-Wire Wire Line
-	950  3950 900  3950
 Connection ~ 800  4050
 Wire Wire Line
-	900  3950 900  4200
-Wire Wire Line
 	800  4200 800  4050
 Wire Wire Line
-	800  4050 900  4050
+	800  4050 1150 4050
 Connection ~ 900  4050
 Wire Wire Line
@@
 	4700 5100 2050 5100
 Wire Wire Line
-	2900 7300 1150 7300
+	1150 7300 3200 7300
 Wire Wire Line
 	1150 7300 1150 6050
@@
 Connection ~ 1600 5950
 Wire Wire Line
-	1150 5850 1700 5850
+	1150 5850 2250 5850
 Wire Wire Line
 	1700 5850 1700 5750
@@
 Wire Wire Line
 	2050 5100 2050 5450
-$Comp
-L GND-RESCUE-fanctl #PWR?
-U 1 1 566DB645
-P 600 5200
-F 0 "#PWR?" H 600 5200 30  0001 C CNN
-F 1 "GND" H 600 5130 30  0001 C CNN
-F 2 "" H 600 5200 60  0001 C CNN
-F 3 "" H 600 5200 60  0001 C CNN
-	1    600  5200
-	-1   0    0    1
-$EndComp
 $Comp
 L ZENER-RESCUE-fanctl D?
@@
 $EndComp
 $Comp
-L GND-RESCUE-fanctl #PWR?
-U 1 1 566B2BF8
-P 900 3950
-F 0 "#PWR?" H 900 3700 50  0001 C CNN
-F 1 "GND" H 900 3800 50  0000 C CNN
-F 2 "" H 900 3950 60  0001 C CNN
-F 3 "" H 900 3950 60  0001 C CNN
-	1    900  3950
-	0    -1   -1   0
-$EndComp
-$Comp
 L Q_PMOS_SDG Q0
 U 1 1 566B3055
@@
 	1    0    0    -1
 $EndComp
+Connection ~ 2900 7300
+$Comp
+L C C0
+U 1 1 5675FD6B
+P 2100 7050
+F 0 "C0" H 2125 7150 50  0000 L CNN
+F 1 "0.1uF" H 2125 6950 50  0000 L CNN
+F 2 "" H 2138 6900 50  0000 C CNN
+F 3 "" H 2100 7050 50  0000 C CNN
+	1    2100 7050
+	1    0    0    -1
+$EndComp
+Wire Wire Line
+	2100 7200 2100 7300
+Connection ~ 2100 7300
+$Comp
+L GND #PWR?
+U 1 1 5675FEE2
+P 2100 6800
+F 0 "#PWR?" H 2100 6550 50  0001 C CNN
+F 1 "GND" H 2100 6650 50  0000 C CNN
+F 2 "" H 2100 6800 50  0000 C CNN
+F 3 "" H 2100 6800 50  0000 C CNN
+	1    2100 6800
+	-1   0    0    1
+$EndComp
+Wire Wire Line
+	2100 6800 2100 6900
+Wire Wire Line
+	900  4050 900  4200
+Wire Wire Line
+	1150 4050 1150 5350
+Wire Wire Line
+	750  5350 1700 5350
+NoConn ~ 1150 5750
+Wire Wire Line
+	2250 5150 4600 5150
+Wire Wire Line
+	4600 5150 4600 5400
+Connection ~ 1700 5850
+$Comp
+L R R?
+U 1 1 56769747
+P 2250 5600
+F 0 "R?" V 2330 5600 50  0000 C CNN
+F 1 "R" V 2250 5600 50  0000 C CNN
+F 2 "" V 2180 5600 50  0000 C CNN
+F 3 "" H 2250 5600 50  0000 C CNN
+	1    2250 5600
+	1    0    0    -1
+$EndComp
+Wire Wire Line
+	2250 5450 2250 5150
+Wire Wire Line
+	2250 5850 2250 5750
 $EndSCHEMATC

Commit message: More changes
Parts:
- removed P? (x6): FAN0, symbol CONN_01X04
- added C1: 0.1uF, symbol C
- added C? (x6): C, symbol C
- added FAN0, FAN1, FAN2, FAN3, FAN4, FAN5: 4PIN_FAN, ab2_header:AB2_HDR_M04-1V_CPU_FAN, symbol 4PIN_FAN
- P?: footprint (none) -> ab2_power:AB2_ATX_PSU-4PIN-V
- R2: renamed from R?; value R -> 68
- U0: footprint (none) -> Housings_DIP:DIP-16_W7.62mm
- gave numbers to parts that had none: 3
Connections:
- net +12V: now also C1.2, C?.1, C?.1, C?.1, C?.1, C?.1, C?.1
- net GND: now also C1.1, C?.2, C?.2, C?.2, C?.2, C?.2, C?.2, FAN0.1 (GND), FAN1.1 (GND), FAN2.1 (GND), FAN3.1 (GND), FAN4.1 (GND), FAN5.1 (GND)
- net at JP1.1, Q0.2 (D): now also FAN0.2 (12V)
- net at IC0.15 ((PCINT1/OC1A)PB1), U0.1 (I1): now also FAN0.4 (PWM)
- net at IC0.16 ((PCINT2/OC1B/~SS~)PB2), U0.2 (I2): now also FAN1.4 (PWM)
- net at JP2.1, Q?.2 (D): now also FAN1.2 (12V)
- net at JP3.1, Q?.2 (D): now also FAN2.2 (12V)
- net at JP4.1, Q?.2 (D): now also FAN3.2 (12V)
- net at JP5.1, Q?.2 (D): now also FAN4.2 (12V)
- net at JP6.1, Q?.2 (D): now also FAN5.2 (12V)
- no-connect marks 2 -> 4

Commit message: Started PSB layout
Parts:
- removed C? (x5): C, symbol C
- removed JP1, JP2, JP3, JP4, JP5, JP6: JUMPER, symbol JUMPER
- removed Q? (x5): Q_PMOS_SDG, symbol Q_PMOS_SDG
- removed R? (x10): R, symbol R
- added C3, C4, C5, C6, C7: 0.1uF, Capacitors_ThroughHole:C_Disc_D3_P2.5, symbol C
- added C8, C9: 22pF, Capacitors_ThroughHole:C_Disc_D3_P2.5, symbol C
- added JP1, JP2, JP3, JP4, JP5, JP6: JUMPER3, Pin_Headers:Pin_Header_Straight_1x03, symbol JUMPER3
- added Q1, Q2, Q3, Q4, Q5: Q_PMOS_SDG, Power_Integrations:TO-220, symbol Q_PMOS_SDG
- added R10, R11, R12, R13, R14, R15, R5, R6, R7, R8, R9: R, Resistors_ThroughHole:Resistor_Horizontal_RM10mm, symbol R
- added Y0: Crystal, Crystals:Crystal_HC49-U_Vertical, symbol Crystal
- C0, C1: footprint (none) -> Capacitors_ThroughHole:C_Disc_D3_P2.5
- C2: renamed from C?; value C -> 0.1uF; footprint (none) -> Capacitors_ThroughHole:C_Disc_D3_P2.5
- D0, D1: footprint (none) -> Diodes_ThroughHole:Diode_DO-35_SOD27_Horizontal_RM10
- IC0: footprint DIL28 -> Housings_DIP:DIP-28_W7.62mm
- JP0: footprint (none) -> Pin_Headers:Pin_Header_Straight_1x02
- Q0: footprint (none) -> Power_Integrations:TO-220
- R0, R1, R2: footprint (none) -> Resistors_ThroughHole:Resistor_Horizontal_RM10mm
- R3, R4: renamed from R?; footprint (none) -> Resistors_ThroughHole:Resistor_Horizontal_RM10mm
- USB0: renamed from P?; footprint (none) -> Connect:USB_B
- gave numbers to parts that had none: 1
Connections:
- net +12V: now also PWR0.1 (P1), C3.1, C4.1, C5.1, C6.1, C7.1, JP1.2, JP2.2, JP3.2, JP4.2, JP5.2, JP6.2; no longer Q0.1 (S), R3.2
- net GND: now also D1.1 (A), IC0.8 (GND), PWR0.2 (P2), PWR0.3 (P3), USB0.5 (shield), C3.2, C4.2, C5.2, C6.2, C7.2, C8.2, C9.2
- net at FAN0.2 (12V), Q0.2 (D): now also JP1.1
- net at IC0.1 ((PCINT14/~RESET~)PC6), JP0.1: now also R15.2
- net XTA2: now reaches IC0.10 ((PCINT7/XTAL2/TOSC2)PB7)
- net XTA2: now also C9.1, Y0.2
- net PWM4: now reaches IC0.11 ((PCINT21/OC0B/T1)PD5), U0.5 (I5)
- net PWM5: now reaches IC0.12 ((PCINT22/OC0A/AIN0)PD6), U0.6 (I6)
- net PWM0: now reaches FAN0.4 (PWM), IC0.15 ((PCINT1/OC1A)PB1), U0.1 (I1)
- net PWM0: now also FAN1.4 (PWM), FAN2.4 (PWM), FAN3.4 (PWM), FAN4.4 (PWM), FAN5.4 (PWM)
- net PWM1: now reaches IC0.16 ((PCINT2/OC1B/~SS~)PB2), U0.2 (I2)
- net PWM1: no longer FAN1.4 (PWM)
- net PWM2: now reaches IC0.17 ((PCINT3/OC2A/MOSI)PB3), U0.3 (I3)
- net TACH0: now reaches IC0.18 ((PCINT4/MISO)PB4)
- net TACH0: now also FAN0.3 (TACH), FAN1.3 (TACH), FAN2.3 (TACH), FAN3.3 (TACH), FAN4.3 (TACH), FAN5.3 (TACH)
- net TACH1: now reaches IC0.19 ((PCINT5/SCK)PB5)
- net +5V: now reaches C0.2, IC0.20 (AVCC), IC0.7 (VCC), R0.2, USB0.1 (VCC)
- net +5V: now also R15.1
- net TACH2: now reaches IC0.23 ((PCINT8/ADC0)PC0)
- net TACH3: now reaches IC0.24 ((PCINT9/ADC1)PC1)
- net TACH4: now reaches IC0.25 ((PCINT10/ADC2)PC2)
- net TACH5: now reaches IC0.26 ((PCINT11/ADC3)PC3)
- net PWM3: now reaches IC0.5 ((PCINT19/OC2B/INT1)PD3), U0.4 (I4)
- net XTA1: now reaches IC0.9 ((PCINT6/XTAL1/TOSC1)PB6)
- net XTA1: now also C8.1, Y0.1
- net at U0.11 (O6): now also R14.2
- net at U0.12 (O5): now also R12.2
- net at U0.13 (O4): now also R10.2
- net at U0.14 (O3): now also R8.2
- net at U0.15 (O2): now also R6.2
- net at FAN1.2 (12V): now also JP2.1, Q1.2 (D)
- net at FAN2.2 (12V): now also JP3.1, Q2.2 (D)
- net at FAN3.2 (12V): now also JP4.1, Q3.2 (D)
- net at FAN4.2 (12V): now also JP5.1, Q4.2 (D)
- net at FAN5.2 (12V): now also JP6.1, Q5.2 (D)
- new net: JP1.3, Q0.1 (S), R3.2
- new net: JP2.3, Q1.1 (S), R5.2
- new net: Q1.3 (G), R5.1, R6.1
- new net: JP3.3, Q2.1 (S), R7.2
- new net: Q2.3 (G), R7.1, R8.1
- new net: JP4.3, Q3.1 (S), R9.2
- new net: Q3.3 (G), R10.1, R9.1
- new net: JP5.3, Q4.1 (S), R11.2
- new net: Q4.3 (G), R11.1, R12.1
- new net: JP6.3, Q5.1 (S), R13.2
- new net: Q5.3 (G), R13.1, R14.1
- no-connect marks 4 -> 11
Other:
- moved on the sheet: C0, C2, FAN0, IC0, JP0, Q0, R3, R4

Commit message: PCB pretty much done, I hope
Parts:
- added I2C0: I2C, Pin_Headers:Pin_Header_Straight_1x03, symbol CONN_01X03
Connections:
- net GND: now also D0.1 (A), I2C0.3 (P3)
- net PWM0: now also IC0.5 ((PCINT19/OC2B/INT1)PD3); no longer FAN1.4 (PWM), FAN2.4 (PWM), FAN3.4 (PWM), FAN4.4 (PWM), FAN5.4 (PWM), IC0.15 ((PCINT1/OC1A)PB1)
- net PWM1: now also FAN1.4 (PWM), IC0.17 ((PCINT3/OC2A/MOSI)PB3); no longer IC0.16 ((PCINT2/OC1B/~SS~)PB2)
- net PWM2: now also FAN2.4 (PWM), IC0.16 ((PCINT2/OC1B/~SS~)PB2); no longer IC0.17 ((PCINT3/OC2A/MOSI)PB3)
- net PWM3: now also FAN3.4 (PWM), IC0.12 ((PCINT22/OC0A/AIN0)PD6), U0.6 (I6); no longer IC0.5 ((PCINT19/OC2B/INT1)PD3), U0.4 (I4)
- net PWM4: now also FAN4.4 (PWM)
- net PWM5: now also FAN5.4 (PWM), IC0.15 ((PCINT1/OC1A)PB1), U0.4 (I4); no longer IC0.12 ((PCINT22/OC0A/AIN0)PD6), U0.6 (I6)
- net TACH0: now also IC0.26 ((PCINT11/ADC3)PC3); no longer FAN1.3 (TACH), FAN2.3 (TACH), FAN3.3 (TACH), FAN4.3 (TACH), FAN5.3 (TACH), IC0.18 ((PCINT4/MISO)PB4)
- net TACH1: now also FAN1.3 (TACH), IC0.25 ((PCINT10/ADC2)PC2); no longer IC0.19 ((PCINT5/SCK)PB5)
- net TACH2: now also FAN2.3 (TACH), IC0.24 ((PCINT9/ADC1)PC1); no longer IC0.23 ((PCINT8/ADC0)PC0)
- net TACH3: now also FAN3.3 (TACH), IC0.18 ((PCINT4/MISO)PB4); no longer IC0.24 ((PCINT9/ADC1)PC1)
- net TACH4: now also FAN4.3 (TACH), IC0.13 ((PCINT23/AIN1)PD7); no longer IC0.25 ((PCINT10/ADC2)PC2)
- net TACH5: now also FAN5.3 (TACH), IC0.14 ((PCINT0/CLKO/ICP1)PB0); no longer IC0.26 ((PCINT11/ADC3)PC3)
- net at IC0.27 ((PCINT12/SDA/ADC4)PC4): now also I2C0.1 (P1)
- net at IC0.28 ((PCINT13/SCL/ADC5)PC5): now also I2C0.2 (P2)
- net PWMO3: now reaches U0.11 (O6)
- net PWMO3: now also R10.2; no longer R14.2
- net PWMO4: now reaches R12.2, U0.12 (O5)
- net PWMO5: now reaches U0.13 (O4)
- net PWMO5: now also R14.2; no longer R10.2
- net PWMO2: now reaches R8.2, U0.14 (O3)
- net PWMO1: now reaches R6.2, U0.15 (O2)
- net PWMO0: now reaches R4.2, U0.16 (O1)
- no-connect marks 11 -> 9

Commit message: Some changes and gerber and drill files
Parts:
- added F0: FUSE, Resistors_ThroughHole:Resistor_Horizontal_RM10mm, symbol FUSE
- D0, D1: Voltage (none) -> 3.6
- Q5: Manufacturer (none) -> Fairchild; Part no (none) -> FQP17P06
- R10, R11, R12, R13, R14, R15, R3, R4, R5, R6, R7, R8, R9: value R -> 10k
Connections:
- net +12V: now also F0.1; no longer PWR0.1 (P1)
- net at PWR0.4 (P4): now also F0.2
Changed lines of the file:
@@
 F 2 "Diodes_ThroughHole:Diode_DO-35_SOD27_Horizontal_RM10" H 1400 5550 60  0001 C CNN
 F 3 "" H 1400 5550 60  0001 C CNN
+F 4 "3.6" H 1400 5550 60  0001 C CNN "Voltage"
 	1    1400 5550
 	0    1    1    0
@@
 F 2 "Diodes_ThroughHole:Diode_DO-35_SOD27_Horizontal_RM10" H 1700 5550 60  0001 C CNN
 F 3 "" H 1700 5550 60  0001 C CNN
+F 4 "3.6" H 1700 5550 60  0001 C CNN "Voltage"
 	1    1700 5550
 	0    1    1    0
@@
 F 3 "" H 850 4400 60  0001 C CNN
 	1    850  4400
-	0    -1   1    0
+	0    1    1    0
 $EndComp
 $Comp
@@
 P 1700 1700
 F 0 "R3" V 1780 1700 50  0000 C CNN
-F 1 "R" V 1700 1700 50  0000 C CNN
+F 1 "10k" V 1700 1700 50  0000 C CNN
 F 2 "Resistors_ThroughHole:Resistor_Horizontal_RM10mm" H 1630 1700 50  0001 C CNN
 F 3 "" H 1700 1700 50  0000 C CNN
@@
 P 1850 2250
 F 0 "R4" V 1930 2250 50  0000 C CNN
-F 1 "R" V 1850 2250 50  0000 C CNN
+F 1 "10k" V 1850 2250 50  0000 C CNN
 F 2 "Resistors_ThroughHole:Resistor_Horizontal_RM10mm" H 1780 2250 50  0001 C CNN
 F 3 "" H 1850 2250 50  0000 C CNN
@@
 L +12V #PWR04
 U 1 1 567B9621
-P 700 3900
-F 0 "#PWR04" H 700 3750 50  0001 C CNN
-F 1 "+12V" H 700 4040 50  0000 C CNN
-F 2 "" H 700 3900 50  0000 C CNN
-F 3 "" H 700 3900 50  0000 C CNN
-	1    700  3900
+P 700 3600
+F 0 "#PWR04" H 700 3450 50  0001 C CNN
+F 1 "+12V" H 700 3740 50  0000 C CNN
+F 2 "" H 700 3600 50  0000 C CNN
+F 3 "" H 700 3600 50  0000 C CNN
+	1    700  3600
 	1    0    0    -1
 $EndComp
@@
 Wire Wire Line
 	2050 1250 1700 1250
-Wire Wire Line
-	700  3900 700  4200
 Wire Wire Line
 	3200 7650 3200 7600
@@
 P 4750 4700
 F 0 "R15" V 4830 4700 50  0000 C CNN
-F 1 "R" V 4750 4700 50  0000 C CNN
+F 1 "10k" V 4750 4700 50  0000 C CNN
 F 2 "Resistors_ThroughHole:Resistor_Horizontal_RM10mm" H 4680 4700 50  0001 C CNN
 F 3 "" H 4750 4700 50  0000 C CNN
@@
 P 3300 1700
 F 0 "R5" V 3380 1700 50  0000 C CNN
-F 1 "R" V 3300 1700 50  0000 C CNN
+F 1 "10k" V 3300 1700 50  0000 C CNN
 F 2 "Resistors_ThroughHole:Resistor_Horizontal_RM10mm" H 3230 1700 50  0001 C CNN
 F 3 "" H 3300 1700 50  0000 C CNN
@@
 P 3450 2250
 F 0 "R6" V 3530 2250 50  0000 C CNN
-F 1 "R" V 3450 2250 50  0000 C CNN
+F 1 "10k" V 3450 2250 50  0000 C CNN
 F 2 "Resistors_ThroughHole:Resistor_Horizontal_RM10mm" H 3380 2250 50  0001 C CNN
 F 3 "" H 3450 2250 50  0000 C CNN
@@
 P 4900 1700
 F 0 "R7" V 4980 1700 50  0000 C CNN
-F 1 "R" V 4900 1700 50  0000 C CNN
+F 1 "10k" V 4900 1700 50  0000 C CNN
 F 2 "Resistors_ThroughHole:Resistor_Horizontal_RM10mm" H 4830 1700 50  0001 C CNN
 F 3 "" H 4900 1700 50  0000 C CNN
@@
 P 5050 2250
 F 0 "R8" V 5130 2250 50  0000 C CNN
-F 1 "R" V 5050 2250 50  0000 C CNN
+F 1 "10k" V 5050 2250 50  0000 C CNN
 F 2 "Resistors_ThroughHole:Resistor_Horizontal_RM10mm" H 4980 2250 50  0001 C CNN
 F 3 "" H 5050 2250 50  0000 C CNN
@@
 P 6500 1700
 F 0 "R9" V 6580 1700 50  0000 C CNN
-F 1 "R" V 6500 1700 50  0000 C CNN
+F 1 "10k" V 6500 1700 50  0000 C CNN
 F 2 "Resistors_ThroughHole:Resistor_Horizontal_RM10mm" H 6430 1700 50  0001 C CNN
 F 3 "" H 6500 1700 50  0000 C CNN
@@
 P 6650 2250
 F 0 "R10" V 6730 2250 50  0000 C CNN
-F 1 "R" V 6650 2250 50  0000 C CNN
+F 1 "10k" V 6650 2250 50  0000 C CNN
 F 2 "Resistors_ThroughHole:Resistor_Horizontal_RM10mm" H 6580 2250 50  0001 C CNN
 F 3 "" H 6650 2250 50  0000 C CNN
@@
 P 8100 1700
 F 0 "R11" V 8180 1700 50  0000 C CNN
-F 1 "R" V 8100 1700 50  0000 C CNN
+F 1 "10k" V 8100 1700 50  0000 C CNN
 F 2 "Resistors_ThroughHole:Resistor_Horizontal_RM10mm" H 8030 1700 50  0001 C CNN
 F 3 "" H 8100 1700 50  0000 C CNN
@@
 P 8250 2250
 F 0 "R12" V 8330 2250 50  0000 C CNN
-F 1 "R" V 8250 2250 50  0000 C CNN
+F 1 "10k" V 8250 2250 50  0000 C CNN
 F 2 "Resistors_ThroughHole:Resistor_Horizontal_RM10mm" H 8180 2250 50  0001 C CNN
 F 3 "" H 8250 2250 50  0000 C CNN
@@
 F 2 "Power_Integrations:TO-220" H 9500 1500 60  0001 C CNN
 F 3 "" H 9500 1500 60  0001 C CNN
+F 4 "Fairchild" H 9500 1500 60  0001 C CNN "Manufacturer"
+F 5 "FQP17P06" H 9500 1500 60  0001 C CNN "Part no"
 	1    9500 1500
 	-1   0    0    -1
@@
 P 9700 1700
 F 0 "R13" V 9780 1700 50  0000 C CNN
-F 1 "R" V 9700 1700 50  0000 C CNN
+F 1 "10k" V 9700 1700 50  0000 C CNN
 F 2 "Resistors_ThroughHole:Resistor_Horizontal_RM10mm" H 9630 1700 50  0001 C CNN
 F 3 "" H 9700 1700 50  0000 C CNN
@@
 P 9850 2250
 F 0 "R14" V 9930 2250 50  0000 C CNN
-F 1 "R" V 9850 2250 50  0000 C CNN
+F 1 "10k" V 9850 2250 50  0000 C CNN
 F 2 "Resistors_ThroughHole:Resistor_Horizontal_RM10mm" H 9780 2250 50  0001 C CNN
 F 3 "" H 9850 2250 50  0000 C CNN
@@
 NoConn ~ 3400 5700
 Connection ~ 1400 5350
+$Comp
+L FUSE F0
+U 1 1 567FB319
+P 700 3900
+F 0 "F0" H 800 3950 50  0000 C CNN
+F 1 "FUSE" H 600 3850 50  0000 C CNN
+F 2 "Resistors_ThroughHole:Resistor_Horizontal_RM10mm" H 700 3900 50  0001 C CNN
+F 3 "" H 700 3900 50  0000 C CNN
+F 4 "10A" H 700 3900 60  0001 C CNN "Amp"
+	1    700  3900
+	0    1    1    0
+$EndComp
+Wire Wire Line
+	700  4200 700  4150
+Wire Wire Line
+	700  3650 700  3600
 $EndSCHEMATC
