File: hw/fanctl.kicad_pcb (KiCad board)
At the start: 2 copper layers, 101.6 x 59.7 mm, 52 parts, among them IC0 ATMEGA168PA-P, Q0 Q_PMOS_SDG, Q1 Q_PMOS_SDG, Q2 Q_PMOS_SDG, Q3 Q_PMOS_SDG, Q4 Q_PMOS_SDG, Q5 Q_PMOS_SDG, U0 ULN2003A, Y0 Crystal

Commit message: PCB pretty much done, I hope
Parts:
- added I2C0: I2C, Pin_Headers:Pin_Header_Straight_1x03, F.Cu at (62.2, 104.1)
- moved C8 19.0 mm to (102.9, 128.3), turned to 180 degrees
- moved C9 14.0 mm to (118.1, 128.3), turned to 0 degrees
- moved C1 8.98 mm to (124.5, 97.8), turned to 180 degrees
- moved R13 8.52 mm to (137.2, 123.2)
- moved R14 3.59 mm to (137.2, 127.0)
- moved C0 2.54 mm to (105.4, 123.2)
- moved IC0 2.54 mm to (87.6, 119.4)
- moved Y0 2.54 mm to (110.5, 128.3)
- moved C7 1.27 mm to (135.9, 116.8)
- moved JP1 1.27 mm to (69.8, 88.9)
- moved JP2 1.27 mm to (92.7, 88.9)
- moved JP3 1.27 mm to (115.6, 88.9)
- moved JP4 1.27 mm to (139.7, 88.9)
- moved Q0 1.27 mm to (76.2, 83.8)
- moved Q1 1.27 mm to (99.1, 83.8)
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Connections:
- net Net-(R12-Pad2) renamed PWMO4
- net Net-(R4-Pad2) renamed PWMO0
- net Net-(R6-Pad2) renamed PWMO1
- net Net-(R8-Pad2) renamed PWMO2
- D0 pad 1: Net-(D0-Pad1) -> GND
- FAN1 pad 3: TACH0 -> TACH1
- FAN1 pad 4: PWM0 -> PWM1
- FAN2 pad 3: TACH0 -> TACH2
- FAN2 pad 4: PWM0 -> PWM2
- FAN3 pad 3: TACH0 -> TACH3
- FAN3 pad 4: PWM0 -> PWM3
- FAN4 pad 3: TACH0 -> TACH4
- FAN4 pad 4: PWM0 -> PWM4
- FAN5 pad 3: TACH0 -> TACH5
- FAN5 pad 4: PWM0 -> PWM5
- IC0 pad 12: PWM5 -> PWM3
- IC0 pad 13: Net-(IC0-Pad13) -> TACH4
- IC0 pad 14: Net-(IC0-Pad14) -> TACH5
- IC0 pad 15: PWM0 -> PWM5
- IC0 pad 16: PWM1 -> PWM2
- IC0 pad 17: PWM2 -> PWM1
- IC0 pad 18: TACH0 -> TACH3
- IC0 pad 19: TACH1 -> Net-(IC0-Pad19)
- IC0 pad 23: TACH2 -> Net-(IC0-Pad23)
- IC0 pad 24: TACH3 -> TACH2
- IC0 pad 25: TACH4 -> TACH1
- IC0 pad 26: TACH5 -> TACH0
- IC0 pad 5: PWM3 -> PWM0
- PWR0 pad 1: Net-(PWR0-Pad1) -> +12V
- PWR0 pad 4: +12V -> Net-(PWR0-Pad4)
- R10 pad 2: Net-(R10-Pad2) -> PWMO3
- R14 pad 2: Net-(R14-Pad2) -> PWMO5
- U0 pad 11: Net-(R14-Pad2) -> PWMO3
- U0 pad 13: Net-(R10-Pad2) -> PWMO5
- U0 pad 4: PWM3 -> PWM5
- U0 pad 6: PWM5 -> PWM3
Routing:
- net +12V: track 34.1 -> 157.9 mm, vias 0 -> 5
- net PWM4: track 0.00 -> 109.8 mm
- net PWM3: track 0.00 -> 84.8 mm, vias 0 -> 2
- net TACH4: track 0.00 -> 72.9 mm, vias 0 -> 5
- net PWM0: track 0.00 -> 70.8 mm, vias 0 -> 7
- net PWM2: track 0.00 -> 65.5 mm
- net PWM5: track 0.00 -> 64.6 mm
- net TACH3: track 0.00 -> 64.5 mm, vias 0 -> 4
- net TACH0: track 0.00 -> 64.4 mm, vias 0 -> 1
- net PWM1: track 0.00 -> 61.8 mm, vias 0 -> 3
- net +5V: track 0.00 -> 60.4 mm
- net TACH2: track 0.00 -> 58.9 mm, vias 0 -> 3
- net Net-(R10-Pad2): track 54.2 -> 0.00 mm
- net PWMO3: track 0.00 -> 49.9 mm
- net PWMO5: track 0.00 -> 49.4 mm
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- added copper zone on F.Cu, net +12V
- added copper zone on B.Cu, net GND
Other:
- outline, holes or cut-outs redrawn
- net class fanpwr added: clearance 0.3, trace_width 1.5, via_dia 2, via_drill 1.5
- board text added: "3-PIN"
- board text added: "4-PIN"
- board text added: "Fanctl v0.1"
- board text added: "GND"
- board text added: "RESET"
- board text added: "SCL"
- board text added: "SDA"
- board text added: "by: Joakim Jalap"
- board text added: "https://github.com/jockej/fanctl"

Commit message: Some changes and gerber and drill files
Parts:
- added F0: FUSE, Resistors_ThroughHole:Resistor_Horizontal_RM10mm, F.Cu at (77.5, 100.3)
- R10, R11, R12, R13, R14, R15, R3, R4, R5, R6, R7, R8, R9: value R -> 10k
- turned PWR0 to 270 degrees
Connections:
- PWR0 pad 1: +12V -> Net-(PWR0-Pad1)
Routing:
- net Net-(F0-Pad2): track 0.00 -> 11.2 mm
- net +12V: track 157.9 -> 150.1 mm
- net PWM0: track 70.8 -> 72.9 mm, vias 7 -> 9
- removed copper zone on F.Cu, net +12V
Other:
- board text added: "Copyright 2015, Joakim Jalap"

Commit message: Some more changes
Parts:
- moved Q0 1.27 mm to (76.2, 85.1)
- moved Q1 1.27 mm to (99.1, 85.1)
- moved Q2 1.27 mm to (121.9, 85.1)
- moved Q3 1.27 mm to (146.1, 85.1)
- moved FAN0 1.27 mm to (76.2, 77.5)
- moved FAN1 1.27 mm to (99.1, 77.5)
- moved FAN2 1.27 mm to (121.9, 77.5)
- moved FAN3 1.27 mm to (146.1, 77.5)
Routing:
- net Net-(FAN3-Pad2): track 22.6 -> 20.8 mm
- net TACH3: track 64.5 -> 63.0 mm
- net TACH2: track 58.9 -> 57.4 mm
- net Net-(JP4-Pad3): track 17.6 -> 16.3 mm
- net Net-(JP1-Pad3): track 19.7 -> 18.4 mm
- net Net-(JP3-Pad3): track 16.1 -> 14.8 mm
- net Net-(JP2-Pad3): track 16.1 -> 14.8 mm
- net TACH0: track 64.4 -> 63.2 mm
- net PWM3: track 84.8 -> 83.6 mm
- net PWM2: track 65.5 -> 64.2 mm
- net Net-(Q0-Pad3): track 10.5 -> 9.94 mm
- net PWM1: track 61.8 -> 61.2 mm
- net PWM0: track 72.9 -> 72.4 mm
